Commit message: camera in gazebo

File: src/capra_gazebo/models/capra6/capra6.urdf (robot description, URDF)
Before this commit: robot capra6, 2 links, 1 joints
Links:
- added link camera, mass 1; collision sphere radius=0.1; visual sphere radius=0.1
- added link pole, mass 1; collision box size=0.05 0.05 1.2; visual box size=0.05 0.05 1.2
Joints:
- added joint joint2: type fixed, parent base_link, child camera, origin xyz=0 0 1.2 rpy=0 0.5 0
- added joint joint4: type fixed, parent base_link, child pole, origin xyz=0 0 0 rpy=0 0 0

Commit message: model 3D a jour

File: src/capra_gazebo/models/capra6/capra6.urdf (robot description, URDF)
Before this commit: robot capra6, 4 links, 3 joints
Links:
- link base_link: geometry collision box size=0.6 0.6 0.2; visual mesh filename=package://capra_gazebo/models/capra6/meshes/capra6.dae
- link camera: geometry collision sphere radius=0.1
- link laser: geometry collision sphere radius=0.1
- link pole: geometry collision box size=0.05 0.05 1.2
