Commit message: config for vision real

File: src/capra_2dnav/models/capra6/capra6.urdf (robot description, URDF)
Before this commit: robot capra6, 4 links, 3 joints
Joints:
- joint joint2: origin xyz=0 0 1.2 rpy=0 0.5 0 -> xyz=0.28 0 1.28 rpy=0 0.5 0

Commit message: testing with noise

File: src/capra_2dnav/models/capra6/capra6.urdf (robot description, URDF)
Before this commit: robot capra6, 4 links, 3 joints
Links:
- link base_link: mass 1 -> 100

Commit message: post tests navigation

File: src/capra_2dnav/models/capra6/capra6.urdf (robot description, URDF)
Before this commit: robot capra6, 4 links, 3 joints
Links:
- added link imu, mass 1; collision sphere radius=0.1
Joints:
- added joint joint5: type fixed, parent base_link, child imu, origin xyz=0 0 0.5 rpy=0 0 0

Commit message: work on imu/kalman, post-tests. J'ai entre autres enlevé les transformations manuelles de tf pour rendre ça automatique dans le urdf

File: src/capra_2dnav/models/capra6/capra6.urdf (robot description, URDF)
Before this commit: robot capra6, 5 links, 4 joints
Joints:
- joint joint5: origin xyz=0 0 0.5 rpy=0 0 0 -> xyz=0 0 0.5 rpy=3.141593 0 1.82079

Commit message: launchfile pour ai de jean luc

File: src/capra_2dnav/models/capra6/capra6.urdf (robot description, URDF)
Before this commit: robot capra6, 5 links, 4 joints
Links:
- removed link imu
- added link imu_robot, mass 1; collision sphere radius=0.1
Joints:
- joint joint5: child imu -> imu_robot; origin xyz=0 0 0.5 rpy=3.141593 0 1.82079 -> xyz=0 0 0.5 rpy=3.141593 0 1.22

Commit message: reoriented camera in gazebo

File: src/capra_2dnav/models/capra6/capra6.urdf (robot description, URDF)
Before this commit: robot capra6, 5 links, 4 joints
Joints:
- joint joint2: origin xyz=0.28 0 1.28 rpy=0 0.5 0 -> xyz=0.28 0 1.28 rpy=0 0.92 0

Commit message: config for demo: many costmap tweaks, made collision box of robot smaller in gazebo

File: src/capra_2dnav/models/capra6/capra6.urdf (robot description, URDF)
Before this commit: robot capra6, 5 links, 4 joints
Links:
- link base_link: geometry collision box size=0.5 0.5 0.2; visual mesh filename=package://capra_gazebo/models/capra6/meshes/capra6.dae
